Commit message: Updated urdf file and gazebo controller plugin

File: src/mirte-ros-packages-mirte-master/mirte_description/urdf/mirte_description.urdf.xacro (robot description, xacro)
@@ -4,20 +4,20 @@
      For more information, please see http://wiki.ros.org/sw_urdf_exporter -->
 <robot
-  name="mirte_description" xmlns:xacro="http://ros.org/wiki/xacro">
+  name="robot_base" xmlns:xacro="http://www.ros.org/wiki/xacro">
   <link
     name="base_link">
     <inertial>
       <origin
-        xyz="-0.00127942588707535 0.0151241102447173 -0.00985810717289011"
-        rpy="0 0 0" />
-      <mass
-        value="1.67774926625852" />
-      <inertia
-        ixx="0.00906343835306296"
-        ixy="8.45553301983081E-07"
-        ixz="-3.93751691212787E-06"
-        iyy="0.0137382930141301"
-        iyz="0.000240421022548359"
-        izz="0.0076615986898399" />
+        xyz="-0.00083266 0.011121 0.0039376"
+        rpy="0 0 0" />
+      <mass
+        value="2.5772" />
+      <inertia
+        ixx="0.013196"
+        ixy="4.1344E-06"
+        ixz="8.4555E-07"
+        iyy="0.010087"
+        iyz="-0.00024042"
+        izz="0.020292" />
     </inertial>
     <visual>
@@ -32,5 +32,5 @@
         name="">
         <color
-          rgba="0.909803921568627 0.443137254901961 0.0313725490196078 1" />
+          rgba="0.52941 0.54902 0.54902 1" />
       </material>
     </visual>
@@ -49,15 +49,15 @@
     <inertial>
       <origin
-        xyz="0.030103 0.034202 0.03996"
+        xyz="6.4107E-05 2.9249E-10 -1.1211E-10"
         rpy="0 0 0" />
       <mass
         value="0.26661" />
       <inertia
-        ixx="8.0546E-05"
-        ixy="2.8056E-15"
-        ixz="1.0884E-14"
+        ixx="9.3196E-05"
+        ixy="-9.6888E-15"
+        ixz="-1.226E-14"
         iyy="8.0546E-05"
-        iyz="1.1213E-14"
-        izz="9.3196E-05" />
+        iyz="1.9673E-15"
+        izz="8.0546E-05" />
     </inertial>
     <visual>
@@ -80,6 +80,6 @@
         rpy="0 0 0" />
       <geometry>
-        <mesh
-          filename="package://mirte_description/meshes/front_left_wheel_link.STL" />
+        <cylinder radius="0.08" length="0.1" />
+        <!-- <mesh filename="package://mirte_description/meshes/front_left_wheel_link.STL" /> -->
       </geometry>
     </collision>
@@ -87,8 +87,8 @@
   <joint
     name="front_left_wheel_joint"
-    type="fixed">
-    <origin
-      xyz="0.16802 -0.050672 -0.07546"
-      rpy="1.5708 0.13151 -1.5708" />
+    type="continuous">
+    <origin
+      xyz="0.128 -0.085 -0.0455"
+      rpy="1.5708 0 0" />
     <parent
       link="base_link" />
@@ -96,5 +96,5 @@
       link="front_left_wheel_link" />
     <axis
-      xyz="0 0 0" />
+      xyz="-1 0 0" />
   </joint>
   <link
@@ -102,15 +102,15 @@
     <inertial>
       <origin
-        xyz="0.030103 0.034202 0.03996"
+        xyz="6.4107E-05 2.1252E-10 -1.9E-10"
         rpy="0 0 0" />
       <mass
         value="0.26661" />
       <inertia
-        ixx="8.0546E-05"
-        ixy="-5.0529E-15"
-        ixz="7.75E-14"
+        ixx="9.3196E-05"
+        ixy="-9.6011E-15"
+        ixz="-7.6917E-14"
         iyy="8.0546E-05"
-        iyz="-1.4708E-15"
-        izz="9.3196E-05" />
+        iyz="-4.5866E-15"
+        izz="8.0546E-05" />
     </inertial>
     <visual>
@@ -133,6 +133,6 @@
         rpy="0 0 0" />
       <geometry>
-        <mesh
-          filename="package://mirte_description/meshes/front_right_wheel_link.STL" />
+        <cylinder radius="0.08" length="0.1" />
+        <!-- <mesh filename="package://mirte_description/meshes/front_right_wheel_link.STL" /> -->
       </geometry>
     </collision>
@@ -140,8 +140,8 @@
   <joint
     name="front_right_wheel_joint"
-    type="fixed">
-    <origin
-      xyz="-0.087976 -0.060085 -0.083647"
-      rpy="1.5708 -0.14316 -1.5708" />
+    type="continuous">
+    <origin
+      xyz="-0.128 -0.085 -0.0455"
+      rpy="1.5708 0 0" />
     <parent
       link="base_link" />
@@ -149,5 +149,58 @@
       link="front_right_wheel_link" />
     <axis
-      xyz="0 0 0" />
+      xyz="-1 0 0" />
+  </joint>
+  <link
+    name="rear_left_wheel_link">
+    <inertial>
+      <origin
+        xyz="6.4107E-05 2.1252E-10 -1.9E-10"
+        rpy="0 0 0" />
+      <mass
+        value="0.26661" />
+      <inertia
+        ixx="9.3196E-05"
+        ixy="-9.5931E-15"
+        ixz="-7.6904E-14"
+        iyy="8.0546E-05"
+        iyz="-4.574E-15"
+        izz="8.0546E-05" />
+    </inertial>
+    <visual>
+      <origin
+        xyz="0 0 0"
+        rpy="0 0 0" />
+      <geometry>
+        <mesh
+          filename="package://mirte_description/meshes/rear_left_wheel_link.STL" />
+      </geometry>
+      <material
+        name="">
+        <color
+          rgba="0.79216 0.81961 0.93333 1" />
+      </material>
+    </visual>
+    <collision>
+      <origin
+        xyz="0 0 0"
+        rpy="0 0 0" />
+      <geometry>
+        <cylinder radius="0.08" length="0.1" />
+        <!-- <mesh filename="package://mirte_description/meshes/rear_left_wheel_link.STL" /> -->
+      </geometry>
+    </collision>
+  </link>
+  <joint
+    name="rear_left_wheel_joint"
+    type="continuous">
+    <origin
+      xyz="0.128 0.085 -0.0455"
+      rpy="1.5708 0 0" />
+    <parent
+      link="base_link" />
+    <child
+      link="rear_left_wheel_link" />
+    <axis
+      xyz="-1 0 0" />
   </joint>
   <link
@@ -155,15 +208,15 @@
     <inertial>
       <origin
-        xyz="0.030103 0.034202 0.03996"
-        rpy="0 0 0" />
-      <mass
-        value="0.26661" />
-      <inertia
-        ixx="8.0546E-05"
-        ixy="1.1771E-15"
-        ixz="9.8191E-15"
-        iyy="8.0546E-05"
-        iyz="1.9298E-14"
-        izz="9.3196E-05" />
+        xyz="6.41072041088764E-05 2.94731093697376E-10 -1.00091462895691E-10"
+        rpy="0 0 0" />
+      <mass
+        value="0.26661498322592" />
+      <inertia
+        ixx="9.3195603896201E-05"
+        ixy="-1.7571315886241E-14"
+        ixz="-1.26520007319569E-14"
+        iyy="8.05457942703286E-05"
+        iyz="4.82091468818614E-17"
+        izz="8.05457942778204E-05" />
     </inertial>
     <visual>
@@ -178,14 +231,14 @@
         name="">
         <color
-          rgba="0.79216 0.81961 0.93333 1" />
-      </material>
-    </visual>
-    <collision>
-      <origin
-        xyz="0 0 0"
-        rpy="0 0 0" />
-      <geometry>
-        <mesh
-          filename="package://mirte_description/meshes/rear_right_wheel_link.STL" />
+          rgba="0.792156862745098 0.819607843137255 0.933333333333333 1" />
+      </material>
+    </visual>
+    <collision>
+      <origin
+        xyz="0 0 0"
+        rpy="0 0 0" />
+      <geometry>
+        <cylinder radius="0.08" length="0.1" />
+        <!-- <mesh filename="package://mirte_description/meshes/rear_right_wheel_link.STL" /> -->
       </geometry>
     </collision>
@@ -193,8 +246,8 @@
   <joint
     name="rear_right_wheel_joint"
-    type="fixed">
-    <origin
-      xyz="-0.087976 0.11997 -0.074702"
-      rpy="1.5708 0.15337 -1.5708" />
+    type="continuous">
+    <origin
+      xyz="-0.128 0.085 -0.0455"
+      rpy="1.5708 0 0" />
     <parent
       link="base_link" />
@@ -202,58 +255,5 @@
       link="rear_right_wheel_link" />
     <axis
-      xyz="0 0 0" />
-  </joint>
-  <link
-    name="rear_left_wheel_link">
-    <inertial>
-      <origin
-        xyz="0.0301029400755673 0.034202366229229 0.039960226040592"
-        rpy="0 0 0" />
-      <mass
-        value="0.266614983226052" />
-      <inertia
-        ixx="8.05457942742895E-05"
-        ixy="-5.04132749678783E-15"
-        ixz="7.74862268226729E-14"
-        iyy="8.05457942724331E-05"
-        iyz="-1.47689691197136E-15"
-        izz="9.31956038947576E-05" />
-    </inertial>
-    <visual>
-      <origin
-        xyz="0 0 0"
-        rpy="0 0 0" />
-      <geometry>
-        <mesh
-          filename="package://mirte_description/meshes/rear_left_wheel_link.STL" />
-      </geometry>
-      <material
-        name="">
-        <color
-          rgba="0.792156862745098 0.819607843137255 0.933333333333333 1" />
-      </material>
-    </visual>
-    <collision>
-      <origin
-        xyz="0 0 0"
-        rpy="0 0 0" />
-      <geometry>
-        <mesh
-          filename="package://mirte_description/meshes/rear_left_wheel_link.STL" />
-      </geometry>
-    </collision>
-  </link>
-  <joint
-    name="rear_left_wheel_joint"
-    type="fixed">
-    <origin
-      xyz="0.16802 0.10992 -0.083647"
-      rpy="1.5708 -0.14316 -1.5708" />
-    <parent
-      link="base_link" />
-    <child
-      link="rear_left_wheel_link" />
-    <axis
-      xyz="0 0 0" />
+      xyz="-1 0 0" />
   </joint>
   <link
@@ -261,15 +261,15 @@
     <inertial>
       <origin
-        xyz="0.0013219 -0.00039201 -0.022261"
-        rpy="0 0 0" />
-      <mass
-        value="0.18813" />
-      <inertia
-        ixx="6.9146E-05"
-        ixy="2.5433E-06"
-        ixz="1.9137E-05"
-        iyy="0.00044907"
-        iyz="-4.2726E-06"
-        izz="0.0004083" />
+        xyz="0.00132191548038025 -0.000392007221992376 -0.0222605569788096"
+        rpy="0 0 0" />
+      <mass
+        value="0.188133920336356" />
+      <inertia
+        ixx="6.91459456639027E-05"
+        ixy="2.54332844338707E-06"
+        ixz="1.91366259472817E-05"
+        iyy="0.000449074814854817"
+        iyz="-4.27256160719624E-06"
+        izz="0.00040830401695793" />
     </inertial>
     <visual>
@@ -284,5 +284,5 @@
         name="">
         <color
-          rgba="0.25098 0.25098 0.25098 1" />
+          rgba="0.250980392156863 0.250980392156863 0.250980392156863 1" />
       </material>
     </visual>
@@ -314,5 +314,5 @@
     <inertial>
       <origin
-        xyz="-3.97749846947626E-10 -0.0183461608911809 -9.54386087724353E-05"
+        xyz="-3.97749846947626E-10 -0.0183461608911809 -9.54386087724342E-05"
         rpy="0 0 0" />
       <mass
@@ -320,6 +320,6 @@
       <inertia
         ixx="3.39518063996325E-05"
-        ixy="-1.6211120950128E-12"
-        ixz="-2.92284267119986E-13"
+        ixy="-1.6211120950645E-12"
+        ixz="-2.92284267223383E-13"
         iyy="4.1935853096105E-05"
         iyz="1.1815579647801E-07"
@@ -364,45 +364,98 @@
   </joint>
   <link
-    name="fron_left_ultrasone_link">
-    <inertial>
-      <origin
-        xyz="-4.3073E-05 0.0036756 -6.9914E-05"
-        rpy="0 0 0" />
-      <mass
-        value="0.0038351" />
-      <inertia
-        ixx="1.5937E-07"
-        ixy="-8.5425E-10"
-        ixz="-3.4091E-09"
-        iyy="7.6875E-07"
-        iyz="2.6506E-09"
-        izz="7.2622E-07" />
-    </inertial>
-    <visual>
-      <origin
-        xyz="0 0 0"
-        rpy="0 0 0" />
-      <geometry>
-        <mesh
-          filename="package://mirte_description/meshes/fron_left_ultrasone_link.STL" />
-      </geometry>
-      <material
-        name="">
-        <color
-          rgba="0.79216 0.81961 0.93333 1" />
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
File: src/mirte-ros-packages-mirte-master/mirte_description/urdf/robot_base.gazebo.xacro (robot description, xacro)
@@ -1,4 +1,4 @@
 <?xml version="1.0"?>
-<robot xmlns:xacro="http://ros.org/wiki/xacro" name="robot_base">
+<robot xmlns:xacro="http://www.ros.org/wiki/xacro" name="robot_base">
    <gazebo reference="base_link">
        <material>Gazebo/Black</material>
@@ -7,7 +7,4 @@
        <mu1>0.0</mu1>
        <mu2>0.0</mu2>
-        <kp value="10000000.0" />
-        <kd value="1.0" />
-        <fdir1 value="1 0 0"/>
        <material>Gazebo/Orange</material>
    </gazebo>
@@ -15,7 +12,4 @@
        <mu1>0.0</mu1>
        <mu2>0.0</mu2>
-        <kp value="10000000.0" />
-        <kd value="1.0" />
-        <fdir1 value="1 0 0"/>
        <material>Gazebo/Orange</material>
    </gazebo>
@@ -23,7 +17,4 @@
        <mu1>0.0</mu1>
        <mu2>0.0</mu2>
-        <kp value="10000000.0" />
-        <kd value="1.0" />
-        <fdir1 value="1 0 0"/>
        <material>Gazebo/Orange</material>
    </gazebo>
@@ -31,7 +22,4 @@
        <mu1>0.0</mu1>
        <mu2>0.0</mu2>
-        <kp value="10000000.0" />
-        <kd value="1.0" />
-        <fdir1 value="1 0 0"/>
        <material>Gazebo/Orange</material>
    </gazebo>
@@ -43,22 +31,20 @@
             <legacyModeNS>false</legacyModeNS>
        </plugin>
-       <!-- <plugin name="gazebo_ros_mecanum_diff_drive" filename="libgazebo_ros_mecanum_drive.so">
+       <!-- <plugin name="mecanum_controller" filename="libgazebo_ros_mecanum_drive.so">
+            <robotNamespace>/</robotNamespace>
             <commandTopic>cmd_vel</commandTopic>
             <odometryTopic>odom</odometryTopic>
             <odometryFrame>odom</odometryFrame>
-            <robotBaseFrame>base_footprint</robotBaseFrame>
+            <robotBaseFrame>base_link</robotBaseFrame>
             <LeftRear>front_left_wheel_joint</LeftRear>
             <LeftFront>front_right_wheel_joint</LeftFront>
             <RightFront>rear_left_wheel_joint</RightFront>
             <RightRear>rear_right_wheel_joint</RightRear>
-            <odometryRate>20</odometryRate>
+            <odometryRate>60</odometryRate>
             <publishWheelTF>true</publishWheelTF>
             <publishWheelJointState>true</publishWheelJointState>
             <WheelTorque>1</WheelTorque>
-            <WheelSeparationW>0.5</WheelSeparationW>
-            <WheelSeparationL>0.6</WheelSeparationL>
             <wheelAccel>5</wheelAccel>
-            <wheelDiameter>0.13</wheelDiameter>
-            <publishOdom>true</publishOdom>
+            <publishOdom>false</publishOdom>
             <isRollerModel>true</isRollerModel>
        </plugin> -->
@@ -70,6 +56,6 @@
             <leftFrontJoint>front_left_wheel_joint</leftFrontJoint>
             <rightFrontJoint>front_right_wheel_joint</rightFrontJoint>
-            <leftRearJoint>back_left_wheel_joint</leftRearJoint>
-            <rightRearJoint>back_right_wheel_joint</rightRearJoint>
+            <leftRearJoint>rear_left_wheel_joint</leftRearJoint>
+            <rightRearJoint>rear_right_wheel_joint</rightRearJoint>
             <odometryRate>60.0</odometryRate>
             <robotBaseFrame>base_link</robotBaseFrame>

Commit message: New features, controller works sometimes

File: src/mirte-ros-packages-mirte-master/mirte_description/urdf/mirte_description.urdf.xacro (robot description, xacro)
@@ -5,4 +5,6 @@
 <robot
   name="robot_base" xmlns:xacro="http://www.ros.org/wiki/xacro">
+  <xacro:property name="radius" value="0.055" />
+  <xacro:property name="length" value="0.05" />
   <link
     name="base_link">
@@ -78,7 +80,7 @@
       <origin
         xyz="0 0 0"
-        rpy="0 0 0" />
-      <geometry>
-        <cylinder radius="0.08" length="0.1" />
+        rpy="0 1.56 0" />
+      <geometry>
+        <cylinder radius="${radius}" length="${length}" />
         <!-- <mesh filename="package://mirte_description/meshes/front_left_wheel_link.STL" /> -->
       </geometry>
@@ -131,7 +133,7 @@
       <origin
         xyz="0 0 0"
-        rpy="0 0 0" />
-      <geometry>
-        <cylinder radius="0.08" length="0.1" />
+        rpy="0 1.56 0" />
+      <geometry>
+        <cylinder radius="${radius}" length="${length}" />
         <!-- <mesh filename="package://mirte_description/meshes/front_right_wheel_link.STL" /> -->
       </geometry>
@@ -184,7 +186,7 @@
       <origin
         xyz="0 0 0"
-        rpy="0 0 0" />
-      <geometry>
-        <cylinder radius="0.08" length="0.1" />
+        rpy="0 1.56 0" />
+      <geometry>
+        <cylinder radius="${radius}" length="${length}" />
         <!-- <mesh filename="package://mirte_description/meshes/rear_left_wheel_link.STL" /> -->
       </geometry>
@@ -237,7 +239,7 @@
       <origin
         xyz="0 0 0"
-        rpy="0 0 0" />
-      <geometry>
-        <cylinder radius="0.08" length="0.1" />
+        rpy="0 1.56 0" />
+      <geometry>
+        <cylinder radius="${radius}" length="${length}" />
         <!-- <mesh filename="package://mirte_description/meshes/rear_right_wheel_link.STL" /> -->
       </geometry>

File: src/mirte-ros-packages-mirte-master/mirte_description/urdf/robot_base.gazebo.xacro (robot description, xacro)
@@ -7,4 +7,6 @@
        <mu1>0.0</mu1>
        <mu2>0.0</mu2>
+       <!-- <kp>1000.0</kp>
+       <kd>0.1</kd>        -->
        <material>Gazebo/Orange</material>
    </gazebo>
@@ -12,4 +14,6 @@
        <mu1>0.0</mu1>
        <mu2>0.0</mu2>
+       <!-- <kp>1000.0</kp>
+       <kd>0.1</kd> -->
        <material>Gazebo/Orange</material>
    </gazebo>
@@ -17,4 +21,6 @@
        <mu1>0.0</mu1>
        <mu2>0.0</mu2>
+       <!-- <kp>1000.0</kp>
+       <kd>0.1</kd>        -->
        <material>Gazebo/Orange</material>
    </gazebo>
@@ -22,4 +28,6 @@
        <mu1>0.0</mu1>
        <mu2>0.0</mu2>
+       <!-- <kp>1000.0</kp>
+       <kd>0.1</kd>        -->
        <material>Gazebo/Orange</material>
    </gazebo>
@@ -61,21 +69,25 @@
             <robotBaseFrame>base_link</robotBaseFrame>
         </plugin> -->
-    <plugin name="diff_drive" filename="libgazebo_ros_diff_drive.so">
-        <dds_domain_id>0</dds_domain_id>
-        <topic_name_twist>cmd_vel</topic_name_twist>
-        <topic_name_odometry>odom</topic_name_odometry>
-        <!-- <topic_name_joint>joint</topic_name_joint> -->
-        <right_front_joint>front_right_wheel_joint</right_front_joint>
-        <right_rear_joint>rear_right_wheel_joint</right_rear_joint>
-        <left_front_joint>front_left_wheel_joint</left_front_joint>
-        <left_rear_joint>rear_left_wheel_joint</left_rear_joint>
-        <!-- <wheel_separation>0.4</wheel_separation>
-        <wheel_diameter>0.15</wheel_diameter> -->
-        <wheel_torque>5.0</wheel_torque>
-        <update_rate>2</update_rate>
-        <covariance_x>0.0001</covariance_x>
-        <covariance_y>0.0001</covariance_y>
-        <covariance_yaw>0.01</covariance_yaw>
-    </plugin>
+      <plugin name="diff_drive_controller" filename="libgazebo_ros_diff_drive.so">
+        <legacyMode>false</legacyMode>
+        <alwaysOn>true</alwaysOn>
+        <updateRate>1000.0</updateRate>
+        <leftJoint>front_left_wheel_joint, rear_left_wheel_joint</leftJoint>
+        <rightJoint>front_right_wheel_joint, rear_right_wheel_joint</rightJoint>
+        <wheelSeparation>0.5</wheelSeparation>
+        <wheelDiameter>0.2</wheelDiameter>
+        <wheelTorque>10</wheelTorque>
+        <publishTf>1</publishTf>
+        <publishOdomTf>1</publishOdomTf>
+        <odometryFrame>map</odometryFrame>
+        <commandTopic>cmd_vel</commandTopic>
+        <odometryTopic>odom</odometryTopic>
+        <robotBaseFrame>base_link</robotBaseFrame>
+        <wheelAcceleration>2.8</wheelAcceleration>
+        <publishWheelJointState>true</publishWheelJointState>
+        <publishWheelTF>false</publishWheelTF>
+        <odometrySource>world</odometrySource>
+        <rosDebugLevel>Debug</rosDebugLevel>
+      </plugin>
    </gazebo>
 </robot>
