Commit message: we did it! we can now drive around in rviz!!! hells yeah!

File: src/mirte-ros-packages-mirte-master/mirte_description/urdf/mirte_description.urdf.xacro (robot description, xacro)
@@ -7,19 +7,21 @@
   <xacro:property name="radius" value="0.055" />
   <xacro:property name="length" value="0.05" />
+  <xacro:property name="wheel_orientation" value="1 0 0" />
+  <xacro:property name="collision_transform" value="0 1.57079632679 1.57079632679" />
   <link
     name="base_link">
     <inertial>
       <origin
-        xyz="-0.00083266 0.011121 0.0039376"
-        rpy="0 0 0" />
-      <mass
-        value="2.5772" />
-      <inertia
-        ixx="0.013196"
-        ixy="4.1344E-06"
-        ixz="8.4555E-07"
-        iyy="0.010087"
-        iyz="-0.00024042"
-        izz="0.020292" />
+        xyz="-0.0111443854086884 -0.000831975562567948 0.00395208351304286"
+        rpy="0 0 0" />
+      <mass
+        value="2.57903452705291" />
+      <inertia
+        ixx="0.010097194230352"
+        ixy="-4.37392111784297E-06"
+        ixz="0.000240822381205553"
+        iyy="0.0132093250149844"
+        iyz="7.47840581370496E-07"
+        izz="0.020314109789297" />
     </inertial>
     <visual>
@@ -34,5 +36,5 @@
         name="">
         <color
-          rgba="0.52941 0.54902 0.54902 1" />
+          rgba="0.529411764705882 0.549019607843137 0.549019607843137 1" />
       </material>
     </visual>
@@ -51,15 +53,15 @@
     <inertial>
       <origin
-        xyz="6.4107E-05 2.9249E-10 -1.1211E-10"
-        rpy="0 0 0" />
-      <mass
-        value="0.26661" />
-      <inertia
-        ixx="9.3196E-05"
-        ixy="-9.6888E-15"
-        ixz="-1.226E-14"
-        iyy="8.0546E-05"
-        iyz="1.9673E-15"
-        izz="8.0546E-05" />
+        xyz="-1.12107309546694E-10 6.41072041116242E-05 2.92491794673388E-10"
+        rpy="0 0 0" />
+      <mass
+        value="0.266614983225976" />
+      <inertia
+        ixx="8.05457942774813E-05"
+        ixy="-1.2260463258983E-14"
+        ixz="1.96734401516725E-15"
+        iyy="9.31956038960016E-05"
+        iyz="-9.68885005345804E-15"
+        izz="8.05457942705124E-05" />
     </inertial>
     <visual>
@@ -74,11 +76,11 @@
         name="">
         <color
-          rgba="0.79216 0.81961 0.93333 1" />
-      </material>
-    </visual>
-    <collision>
-      <origin
-        xyz="0 0 0"
-        rpy="0 1.56 0" />
+          rgba="0.792156862745098 0.819607843137255 0.933333333333333 1" />
+      </material>
+    </visual>
+    <collision>
+      <origin
+        xyz="0 0 0"
+        rpy="${collision_transform}" />
       <geometry>
         <cylinder radius="${radius}" length="${length}" />
@@ -91,6 +93,6 @@
     type="continuous">
     <origin
-      xyz="0.128 -0.085 -0.0455"
-      rpy="1.5708 0 0" />
+      xyz="0.085 0.128 -0.0455"
+      rpy="0 0 0" />
     <parent
       link="base_link" />
@@ -98,5 +100,5 @@
       link="front_left_wheel_link" />
     <axis
-      xyz="-1 0 0" />
+      xyz="0 -1 0" />
   </joint>
   <link
@@ -104,15 +106,15 @@
     <inertial>
       <origin
-        xyz="6.4107E-05 2.1252E-10 -1.9E-10"
-        rpy="0 0 0" />
-      <mass
-        value="0.26661" />
-      <inertia
-        ixx="9.3196E-05"
-        ixy="-9.6011E-15"
-        ixz="-7.6917E-14"
-        iyy="8.0546E-05"
-        iyz="-4.5866E-15"
-        izz="8.0546E-05" />
+        xyz="-1.90001653299632E-10 6.41072041136781E-05 2.12521250597675E-10"
+        rpy="0 0 0" />
+      <mass
+        value="0.266614983226051" />
+      <inertia
+        ixx="8.05457942757E-05"
+        ixy="-7.6916734798387E-14"
+        ixz="-4.58661925987117E-15"
+        iyy="9.31956038947894E-05"
+        iyz="-9.60110972210022E-15"
+        izz="8.05457942710755E-05" />
     </inertial>
     <visual>
@@ -127,11 +129,11 @@
         name="">
         <color
-          rgba="0.79216 0.81961 0.93333 1" />
-      </material>
-    </visual>
-    <collision>
-      <origin
-        xyz="0 0 0"
-        rpy="0 1.56 0" />
+          rgba="0.792156862745098 0.819607843137255 0.933333333333333 1" />
+      </material>
+    </visual>
+    <collision>
+      <origin
+        xyz="0 0 0"
+        rpy="${collision_transform}" />
       <geometry>
         <cylinder radius="${radius}" length="${length}" />
@@ -144,6 +146,6 @@
     type="continuous">
     <origin
-      xyz="-0.128 -0.085 -0.0455"
-      rpy="1.5708 0 0" />
+      xyz="0.085 -0.128 -0.0455"
+      rpy="0 0 0" />
     <parent
       link="base_link" />
@@ -151,5 +153,5 @@
       link="front_right_wheel_link" />
     <axis
-      xyz="-1 0 0" />
+      xyz="0 -1 0" />
   </joint>
   <link
@@ -157,15 +159,15 @@
     <inertial>
       <origin
-        xyz="6.4107E-05 2.1252E-10 -1.9E-10"
-        rpy="0 0 0" />
-      <mass
-        value="0.26661" />
-      <inertia
-        ixx="9.3196E-05"
-        ixy="-9.5931E-15"
-        ixz="-7.6904E-14"
-        iyy="8.0546E-05"
-        iyz="-4.574E-15"
-        izz="8.0546E-05" />
+        xyz="-1.90001639421844E-10 6.41072041137336E-05 2.12521319986614E-10"
+        rpy="0 0 0" />
+      <mass
+        value="0.266614983226051" />
+      <inertia
+        ixx="8.05457942756754E-05"
+        ixy="-7.69042802358516E-14"
+        ixz="-4.57395491293476E-15"
+        iyy="9.31956038947576E-05"
+        iyz="-9.59312925333487E-15"
+        izz="8.05457942710471E-05" />
     </inertial>
     <visual>
@@ -180,11 +182,11 @@
         name="">
         <color
-          rgba="0.79216 0.81961 0.93333 1" />
-      </material>
-    </visual>
-    <collision>
-      <origin
-        xyz="0 0 0"
-        rpy="0 1.56 0" />
+          rgba="0.792156862745098 0.819607843137255 0.933333333333333 1" />
+      </material>
+    </visual>
+    <collision>
+      <origin
+        xyz="0 0 0"
+        rpy="${collision_transform}" />
       <geometry>
         <cylinder radius="${radius}" length="${length}" />
@@ -197,6 +199,6 @@
     type="continuous">
     <origin
-      xyz="0.128 0.085 -0.0455"
-      rpy="1.5708 0 0" />
+      xyz="-0.085 0.128 -0.0455"
+      rpy="0 0 0" />
     <parent
       link="base_link" />
@@ -204,5 +206,5 @@
       link="rear_left_wheel_link" />
     <axis
-      xyz="-1 0 0" />
+      xyz="0 -1 0" />
   </joint>
   <link
@@ -210,15 +212,15 @@
     <inertial>
       <origin
-        xyz="6.41072041088764E-05 2.94731093697376E-10 -1.00091462895691E-10"
+        xyz="-1.00091421262327E-10 6.41072041089319E-05 2.94731093697376E-10"
         rpy="0 0 0" />
       <mass
         value="0.26661498322592" />
       <inertia
-        ixx="9.3195603896201E-05"
-        ixy="-1.7571315886241E-14"
-        ixz="-1.26520007319569E-14"
-        iyy="8.05457942703286E-05"
-        iyz="4.82091468818614E-17"
-        izz="8.05457942778204E-05" />
+        ixx="8.05457942778204E-05"
+        ixy="-1.2652000339339E-14"
+        ixz="4.82096941386991E-17"
+        iyy="9.31956038962011E-05"
+        iyz="-1.75713136841005E-14"
+        izz="8.05457942703287E-05" />
     </inertial>
     <visual>
@@ -239,5 +241,5 @@
       <origin
         xyz="0 0 0"
-        rpy="0 1.56 0" />
+        rpy="${collision_transform}" />
       <geometry>
         <cylinder radius="${radius}" length="${length}" />
@@ -250,6 +252,6 @@
     type="continuous">
     <origin
-      xyz="-0.128 0.085 -0.0455"
-      rpy="1.5708 0 0" />
+      xyz="-0.085 -0.128 -0.0455"
+      rpy="0 0 0" />
     <parent
       link="base_link" />
@@ -257,5 +259,5 @@
       link="rear_right_wheel_link" />
     <axis
-      xyz="-1 0 0" />
+      xyz="0 -1 0" />
   </joint>
   <link
@@ -263,15 +265,15 @@
     <inertial>
       <origin
-        xyz="0.00132191548038025 -0.000392007221992376 -0.0222605569788096"
-        rpy="0 0 0" />
-      <mass
-        value="0.188133920336356" />
-      <inertia
-        ixx="6.91459456639027E-05"
-        ixy="2.54332844338707E-06"
-        ixz="1.91366259472817E-05"
-        iyy="0.000449074814854817"
-        iyz="-4.27256160719624E-06"
-        izz="0.00040830401695793" />
+        xyz="-0.0222605572085065 0.00132191545179521 -0.000392007230496989"
+        rpy="0 0 0" />
+      <mass
+        value="0.188133922243291" />
+      <inertia
+        ixx="0.000408304025984058"
+        ixy="1.91366258287762E-05"
+        ixz="-4.27256164755698E-06"
+        iyy="6.91459464023262E-05"
+        iyz="2.54332903063166E-06"
+        izz="0.00044907482518408" />
     </inertial>
     <visual>
@@ -303,6 +305,6 @@
     type="fixed">
     <origin
-      xyz="0 -0.14666 0.0427"
-      rpy="1.5708 0 0" />
+      xyz="0.14666 0 0.0427"
+      rpy="0 0 0" />
     <parent
       link="base_link" />
@@ -316,5 +318,5 @@
     <inertial>
       <origin
-        xyz="-3.97749846947626E-10 -0.0183461608911809 -9.54386087724342E-05"
+        xyz="-3.97749846947626E-10 -9.54386087724289E-05 -0.0118651639742243"
         rpy="0 0 0" />
       <mass
@@ -322,9 +324,9 @@
       <inertia
         ixx="3.39518063996325E-05"
-        ixy="-1.6211120950645E-12"
-        ixz="-2.92284267223383E-13"
-        iyy="4.1935853096105E-05"
-        iyz="1.1815579647801E-07"
-        izz="3.44778101670497E-05" />
+        ixy="-2.92284267117192E-13"
+        ixz="1.62111209503273E-12"
+        iyy="3.44778101670497E-05"
+        iyz="-1.18155796478011E-07"
+        izz="4.1935853096105E-05" />
     </inertial>
     <visual>
@@ -356,6 +358,6 @@
     type="fixed">
     <origin
-      xyz="0 -0.1005 -0.023"
-      rpy="-1.5708 0 -1.5708" />
+      xyz="0.1005 0 0.0072113"
+      rpy="0 0 0" />
     <parent
       link="base_link" />
@@ -369,5 +371,5 @@
     <inertial>
       <origin
-        xyz="-4.30733527063201E-05 0.00367564883489799 -6.9913657863175E-05"
+        xyz="4.30733527063271E-05 0.00367564883489799 6.9913657863175E-05"
         rpy="0 0 0" />
       <mass
@@ -375,9 +377,9 @@
       <inertia
         ixx="1.59365628586767E-07"
-        ixy="-8.54250314742368E-10"
+        ixy="8.54250314742497E-10"
         ixz="-3.40905422018182E-09"
         iyy="7.6875152346034E-07"
-        iyz="2.65062440645525E-09"
-        izz="7.26221149125633E-07" />
+        iyz="-2.65062440645525E-09"
+        izz="7.26221149125632E-07" />
     </inertial>
     <visual>
@@ -409,6 +411,6 @@
     type="fixed">
     <origin
-      xyz="-0.052978 -0.12028 -0.031"
-      rpy="3.1416 0 -0.29671" />
+      xyz="0.12028 -0.052978 -0.031"
+      rpy="0 0 -1.8675" />
     <parent
       link="base_link" />
@@ -422,5 +424,5 @@
     <inertial>
       <origin
-        xyz="-4.30733527062924E-05 0.00367564883489804 -6.99136578631437E-05"
+        xyz="-4.30733527062924E-05 -0.00367564883489804 6.99136578631437E-05"
         rpy="0 0 0" />
       <mass
@@ -428,9 +430,9 @@
       <inertia
         ixx="1.59365628586768E-07"
-        ixy="-8.54250314742662E-10"
-        ixz="-3.40905422018192E-09"
+        ixy="8.54250314742616E-10"
+        ixz="3.40905422018196E-09"
         iyy="7.68751523460337E-07"
-        iyz="2.65062440645509E-09"
-        izz="7.26221149125629E-07" />
+        iyz="2.65062440645508E-09"
+        izz="7.26221149125628E-07" />
     </inertial>
     <visual>
@@ -462,6 +464,6 @@
     type="fixed">
     <origin
-      xyz="0.052978 -0.12028 -0.031"
-      rpy="3.1416 0 0.29671" />
+      xyz="0.12028 0.052978 -0.031"
+      rpy="0 0 1.8675" />
     <parent
       link="base_link" />
@@ -475,5 +477,5 @@
     <inertial>
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