Commit message: Added slam toolbox and fixed some gazebo settings, also fixed the flag giving it 0 weight and changing the inertia of the mirte

File: src/mirte-ros-packages-mirte-master/mirte_description/urdf/mirte_description.urdf.xacro (robot description, xacro)
@@ -13,15 +13,15 @@
     <inertial>
       <origin
-        xyz="-0.0111443854086884 -0.000831975562567948 0.00395208351304286"
-        rpy="0 0 0" />
-      <mass
-        value="2.57903452705291" />
-      <inertia
-        ixx="0.010097194230352"
-        ixy="-4.37392111784297E-06"
-        ixz="0.000240822381205553"
-        iyy="0.0132093250149844"
-        iyz="7.47840581370496E-07"
-        izz="0.020314109789297" />
+        xyz="-0.00910410219928872 -9.31202386654388E-05 -0.00269627899619879"
+        rpy="0 0 0" />
+      <mass
+        value="2.54161575728203" />
+      <inertia
+        ixx="0.00900908568706438"
+        ixy="-1.49036665189052E-06"
+        ixz="0.000180180089420441"
+        iyy="0.0120513643006957"
+        iyz="-7.98162115966032E-07"
+        izz="0.0202435224080604" />
     </inertial>
     <visual>
@@ -53,14 +53,14 @@
     <inertial>
       <origin
-        xyz="-1.12107309546694E-10 6.41072041116242E-05 2.92491794673388E-10"
+        xyz="-1.12107378935633E-10 6.41072041116797E-05 2.92491780795601E-10"
         rpy="0 0 0" />
       <mass
         value="0.266614983225976" />
       <inertia
-        ixx="8.05457942774813E-05"
+        ixx="8.05457942774812E-05"
         ixy="-1.2260463258983E-14"
-        ixz="1.96734401516725E-15"
-        iyy="9.31956038960016E-05"
-        iyz="-9.68885005345804E-15"
+        ixz="1.9673439489928E-15"
+        iyy="9.31956038960015E-05"
+        iyz="-9.68884941818333E-15"
         izz="8.05457942705124E-05" />
     </inertial>
@@ -85,5 +85,6 @@
       <geometry>
         <cylinder radius="${radius}" length="${length}" />
-        <!-- <mesh filename="package://mirte_description/meshes/front_left_wheel_link.STL" /> -->
+        <!-- <mesh
+          filename="package://mirte_description/meshes/front_left_wheel_link.STL" /> -->
       </geometry>
     </collision>
@@ -93,5 +94,5 @@
     type="continuous">
     <origin
-      xyz="0.085 0.128 -0.0455"
+      xyz="0.085 0.128 -0.0454999999999998"
       rpy="0 0 0" />
     <parent
@@ -100,5 +101,5 @@
       link="front_left_wheel_link" />
     <axis
-      xyz="0 -1 0" />
+      xyz="0 1 0" />
   </joint>
   <link
@@ -106,5 +107,5 @@
     <inertial>
       <origin
-        xyz="-1.90001653299632E-10 6.41072041136781E-05 2.12521250597675E-10"
+        xyz="-1.9000166717742E-10 6.41072041136226E-05 2.1252127835325E-10"
         rpy="0 0 0" />
       <mass
@@ -112,9 +113,9 @@
       <inertia
         ixx="8.05457942757E-05"
-        ixy="-7.6916734798387E-14"
-        ixz="-4.58661925987117E-15"
-        iyy="9.31956038947894E-05"
-        iyz="-9.60110972210022E-15"
-        izz="8.05457942710755E-05" />
+        ixy="-7.69167351689639E-14"
+        ixz="-4.58661949809919E-15"
+        iyy="9.31956038947893E-05"
+        iyz="-9.60111009267714E-15"
+        izz="8.05457942710754E-05" />
     </inertial>
     <visual>
@@ -138,5 +139,6 @@
       <geometry>
         <cylinder radius="${radius}" length="${length}" />
-        <!-- <mesh filename="package://mirte_description/meshes/front_right_wheel_link.STL" /> -->
+        <!-- <mesh
+          filename="package://mirte_description/meshes/front_right_wheel_link.STL" /> -->
       </geometry>
     </collision>
@@ -146,5 +148,5 @@
     type="continuous">
     <origin
-      xyz="0.085 -0.128 -0.0455"
+      xyz="0.085 -0.128 -0.0454999999999999"
       rpy="0 0 0" />
     <parent
@@ -153,5 +155,5 @@
       link="front_right_wheel_link" />
     <axis
-      xyz="0 -1 0" />
+      xyz="0 1 0" />
   </joint>
   <link
@@ -159,14 +161,14 @@
     <inertial>
       <origin
-        xyz="-1.90001639421844E-10 6.41072041137336E-05 2.12521319986614E-10"
+        xyz="-1.90001639421844E-10 6.41072041137336E-05 2.12521299169932E-10"
         rpy="0 0 0" />
       <mass
         value="0.266614983226051" />
       <inertia
-        ixx="8.05457942756754E-05"
-        ixy="-7.69042802358516E-14"
-        ixz="-4.57395491293476E-15"
-        iyy="9.31956038947576E-05"
-        iyz="-9.59312925333487E-15"
+        ixx="8.05457942756755E-05"
+        ixy="-7.6904280182912E-14"
+        ixz="-4.57395497910921E-15"
+        iyy="9.31956038947575E-05"
+        iyz="-9.59312938568377E-15"
         izz="8.05457942710471E-05" />
     </inertial>
@@ -191,5 +193,6 @@
       <geometry>
         <cylinder radius="${radius}" length="${length}" />
-        <!-- <mesh filename="package://mirte_description/meshes/rear_left_wheel_link.STL" /> -->
+        <!-- <mesh
+          filename="package://mirte_description/meshes/rear_left_wheel_link.STL" /> -->
       </geometry>
     </collision>
@@ -199,5 +202,5 @@
     type="continuous">
     <origin
-      xyz="-0.085 0.128 -0.0455"
+      xyz="-0.0849999999999993 0.128 -0.045500000000002"
       rpy="0 0 0" />
     <parent
@@ -206,5 +209,5 @@
       link="rear_left_wheel_link" />
     <axis
-      xyz="0 -1 0" />
+      xyz="0 1 0" />
   </joint>
   <link
@@ -212,5 +215,5 @@
     <inertial>
       <origin
-        xyz="-1.00091421262327E-10 6.41072041089319E-05 2.94731093697376E-10"
+        xyz="-1.00091421262327E-10 6.41072041089319E-05 2.94731128391845E-10"
         rpy="0 0 0" />
       <mass
@@ -218,9 +221,9 @@
       <inertia
         ixx="8.05457942778204E-05"
-        ixy="-1.2652000339339E-14"
-        ixz="4.82096941386991E-17"
-        iyy="9.31956038962011E-05"
-        iyz="-1.75713136841005E-14"
-        izz="8.05457942703287E-05" />
+        ixy="-1.26520007959427E-14"
+        ixz="4.82090522465438E-17"
+        iyy="9.3195603896201E-05"
+        iyz="-1.75713132076445E-14"
+        izz="8.05457942703286E-05" />
     </inertial>
     <visual>
@@ -244,5 +247,6 @@
       <geometry>
         <cylinder radius="${radius}" length="${length}" />
-        <!-- <mesh filename="package://mirte_description/meshes/rear_right_wheel_link.STL" /> -->
+        <!-- <mesh
+          filename="package://mirte_description/meshes/rear_right_wheel_link.STL" /> -->
       </geometry>
     </collision>
@@ -252,5 +256,5 @@
     type="continuous">
     <origin
-      xyz="-0.085 -0.128 -0.0455"
+      xyz="-0.0850000000000007 -0.128 -0.0454999999999994"
       rpy="0 0 0" />
     <parent
@@ -259,5 +263,5 @@
       link="rear_right_wheel_link" />
     <axis
-      xyz="0 -1 0" />
+      xyz="0 1 0" />
   </joint>
   <link
@@ -265,15 +269,15 @@
     <inertial>
       <origin
-        xyz="-0.0222605572085065 0.00132191545179521 -0.000392007230496989"
-        rpy="0 0 0" />
-      <mass
-        value="0.188133922243291" />
-      <inertia
-        ixx="0.000408304025984058"
-        ixy="1.91366258287762E-05"
-        ixz="-4.27256164755698E-06"
-        iyy="6.91459464023262E-05"
-        iyz="2.54332903063166E-06"
-        izz="0.00044907482518408" />
+        xyz="-0.0222605569788096 0.00132191548038024 -0.00039200722199239"
+        rpy="0 0 0" />
+      <mass
+        value="0.188133920336356" />
+      <inertia
+        ixx="0.00040830401695793"
+        ixy="1.91366259472818E-05"
+        ixz="-4.27256160719641E-06"
+        iyy="6.91459456639027E-05"
+        iyz="2.54332844338714E-06"
+        izz="0.000449074814854817" />
     </inertial>
     <visual>
@@ -305,5 +309,5 @@
     type="fixed">
     <origin
-      xyz="0.14666 0 0.0427"
+      xyz="0.146658788505756 0 0.0426999999999987"
       rpy="0 0 0" />
     <parent
@@ -318,5 +322,5 @@
     <inertial>
       <origin
-        xyz="-3.97749846947626E-10 -9.54386087724289E-05 -0.0118651639742243"
+        xyz="-3.97749846947626E-10 -9.543860877243E-05 -0.0118651639742243"
         rpy="0 0 0" />
       <mass
@@ -324,8 +328,8 @@
       <inertia
         ixx="3.39518063996325E-05"
-        ixy="-2.92284267117192E-13"
-        ixz="1.62111209503273E-12"
+        ixy="-2.92284267049194E-13"
+        ixz="1.62111209504698E-12"
         iyy="3.44778101670497E-05"
-        iyz="-1.18155796478011E-07"
+        iyz="-1.1815579647801E-07"
         izz="4.1935853096105E-05" />
     </inertial>
@@ -358,5 +362,5 @@
     type="fixed">
     <origin
-      xyz="0.1005 0 0.0072113"
+      xyz="0.1005 0 0.0072113248654052"
       rpy="0 0 0" />
     <parent
@@ -374,11 +378,11 @@
         rpy="0 0 0" />
       <mass
-        value="0.00383513951999245" />
+        value="0.00383513951999244" />
       <inertia
         ixx="1.59365628586767E-07"
-        ixy="8.54250314742497E-10"
+        ixy="8.54250314742398E-10"
         ixz="-3.40905422018182E-09"
         iyy="7.6875152346034E-07"
-        iyz="-2.65062440645525E-09"
+        iyz="-2.65062440645524E-09"
         izz="7.26221149125632E-07" />
     </inertial>
@@ -411,6 +415,6 @@
     type="fixed">
     <origin
-      xyz="0.12028 -0.052978 -0.031"
-      rpy="0 0 -1.8675" />
+      xyz="0.120282421780502 -0.05297775289576 -0.031"
+      rpy="0 0 -1.86750229963393" />
     <parent
       link="base_link" />
@@ -430,8 +434,8 @@
       <inertia
         ixx="1.59365628586768E-07"
-        ixy="8.54250314742616E-10"
-        ixz="3.40905422018196E-09"
+        ixy="8.54250314742599E-10"
+        ixz="3.40905422018193E-09"
         iyy="7.68751523460337E-07"
-        iyz="2.65062440645508E-09"
+        iyz="2.65062440645509E-09"
         izz="7.26221149125628E-07" />
     </inertial>
@@ -464,6 +468,6 @@
     type="fixed">
     <origin
-      xyz="0.12028 0.052978 -0.031"
-      rpy="0 0 1.8675" />
+      xyz="0.120282421780502 0.05297775289576 -0.031"
+      rpy="0 0 1.86750229963393" />
     <parent
       link="base_link" />
@@ -477,5 +481,5 @@
     <inertial>
       <origin
-        xyz="4.30733527062716E-05 0.00367564883489802 6.99136578631784E-05"
+        xyz="4.30733527062785E-05 0.00367564883489802 6.99136578631784E-05"
         rpy="0 0 0" />
       <mass
@@ -483,9 +487,9 @@
       <inertia
         ixx="1.59365628586767E-07"
-        ixy="8.54250314742189E-10"
+        ixy="8.54250314742249E-10"
         ixz="-3.40905422018205E-09"
-        iyy="7.6875152346034E-07"
-        iyz="-2.65062440645534E-09"
-        izz="7.26221149125632E-07" />
+        iyy="7.68751523460339E-07"
+        iyz="-2.65062440645536E-09"
+        izz="7.26221149125631E-07" />
     </inertial>
     <visual>
@@ -517,6 +521,6 @@
     type="fixed">
     <origin
-      xyz="-0.11919 0.056561 -0.031"
-      rpy="0 0 1.2741" />
+      xyz="-0.119187021096338 0.0565606470918482 -0.0309999999999999"
+      rpy="0 0 1.27409035395586" />
     <parent
       link="base_link" />
@@ -536,8 +540,8 @@
       <inertia
         ixx="1.59365628586768E-07"
-        ixy="8.54250314743036E-10"
-        ixz="-3.40905422018172E-09"
+        ixy="8.54250314743049E-10"
+        ixz="-3.40905422018174E-09"
         iyy="7.68751523460337E-07"
-        iyz="-2.65062440645517E-09"
+        iyz="-2.65062440645516E-09"
         izz="7.26221149125628E-07" />
     </inertial>
@@ -576,4 +580,57 @@
     <child
       link="rear_right_ultrasound_link" />
+    <axis
+      xyz="0 0 0" />
+  </joint>
+  <link
+    name="flag_link">
+    <inertial>
+      <origin
+        xyz="-0.024941 -0.00081775 0.13848"
+        rpy="0 0 0" />
+      <mass
+        value="0" />
+      <inertia
+        ixx="0.0010881"
+        ixy="-2.8836E-06"
+        ixz="6.0642E-05"
+        iyy="0.001158"
+        iyz="1.546E-06"
+        izz="7.0587E-05" />
+    </inertial>
+    <visual>
+      <origin
+        xyz="0 0 0"
+        rpy="0 0 0" />
+      <geometry>
+        <mesh
+          filename="package://mirte_description/meshes/flag_link.STL" />
+      </geometry>
+      <material
+        name="">
+        <color
+          rgba="0.79608 0.82353 0.93725 1" />
+      </material>
+    </visual>
+    <collision>
+      <origin
+        xyz="0 0 0"
+        rpy="0 0 0" />
+      <geometry>
+        <mesh
+          filename="package://mirte_description/meshes/flag_link.STL" />
+      </geometry>
+    </collision>
+  </link>
+  <joint
+    name="flag_joint"
+    type="fixed">
+    <origin
+      xyz="-0.12479 -0.0502 0.31705"
+      rpy="0 0 0" />
+    <parent
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
File: src/mirte-ros-packages-mirte-master/mirte_description/urdf/robot_base.gazebo.xacro (robot description, xacro)
@@ -1,10 +1,12 @@
 <?xml version="1.0"?>
 <robot xmlns:xacro="http://www.ros.org/wiki/xacro" name="robot_base">
+  <xacro:property name="set_mu1" value="0.5" />
+  <xacro:property name="set_mu2" value="0.5" />
    <gazebo reference="base_link">
        <material>Gazebo/Black</material>
    </gazebo>
    <gazebo reference="front_left_wheel_link">
-       <mu1>0.0</mu1>
-       <mu2>0.0</mu2>
+       <mu1>${set_mu1}</mu1>
+       <mu2>${set_mu2}</mu2>
        <!-- <kp>1000.0</kp>
        <kd>0.1</kd>        -->
@@ -12,6 +14,6 @@
    </gazebo>
    <gazebo reference="rear_left_wheel_link">
-       <mu1>0.0</mu1>
-       <mu2>0.0</mu2>
+       <mu1>${set_mu1}</mu1>
+       <mu2>${set_mu2}</mu2>
        <!-- <kp>1000.0</kp>
        <kd>0.1</kd> -->
@@ -19,6 +21,6 @@
    </gazebo>
    <gazebo reference="front_right_wheel_link">
-       <mu1>0.0</mu1>
-       <mu2>0.0</mu2>
+       <mu1>${set_mu1}</mu1>
+       <mu2>${set_mu2}</mu2>
        <!-- <kp>1000.0</kp>
        <kd>0.1</kd>        -->
@@ -26,10 +28,45 @@
    </gazebo>
    <gazebo reference="rear_right_wheel_link">
-       <mu1>0.0</mu1>
-       <mu2>0.0</mu2>
+       <mu1>${set_mu1}</mu1>
+       <mu2>${set_mu2}</mu2>
        <!-- <kp>1000.0</kp>
        <kd>0.1</kd>        -->
        <material>Gazebo/Orange</material>
    </gazebo>
+<gazebo reference="lidar_link">
+        <sensor type="ray" name="lidar_sensor">
+        <pose>0 0 0 0 0 0</pose>
+        <visualize>true</visualize>
+        <update_rate>50</update_rate>
+        <ray>
+            <scan>
+            <horizontal>
+                <samples>719</samples>
+                <resolution>1</resolution>
+                <min_angle>-3.1415</min_angle>
+                <max_angle>3.1415</max_angle>
+            </horizontal>
+            </scan>
+            <range>
+            <min>0.30</min>
+            <max>10.0</max>
+            <resolution>0.01</resolution>
+            </range>
+            <noise>
+            <type>gaussian</type>
+            <!-- Noise parameters based on published spec for Hokuyo laser
+                achieving "+-30mm" accuracy at range < 10m.  A mean of 0.0m and
+                stddev of 0.01m will put 99.7% of samples within 0.03m of the true
+                reading. -->
+            <mean>0.0</mean>
+            <stddev>0.01</stddev>
+            </noise>
+        </ray>
+        <plugin name="lidar_sensor_controller" filename="libgazebo_ros_laser.so">
+            <topicName>/scan</topicName>
+            <frameName>lidar_link</frameName>
+        </plugin>
+        </sensor>
+</gazebo>
 <!--######################################################################-->
    <gazebo>
@@ -72,10 +109,10 @@
         <legacyMode>false</legacyMode>
         <alwaysOn>true</alwaysOn>
-        <updateRate>1000.0</updateRate>
+        <updateRate>50.0</updateRate>
         <leftJoint>front_left_wheel_joint, rear_left_wheel_joint</leftJoint>
         <rightJoint>front_right_wheel_joint, rear_right_wheel_joint</rightJoint>
-        <wheelSeparation>0.5</wheelSeparation>
-        <wheelDiameter>0.2</wheelDiameter>
-        <wheelTorque>10</wheelTorque>
+        <wheelSeparation>0.256</wheelSeparation>
+        <wheelDiameter>0.102</wheelDiameter>
+        <wheelTorque>1</wheelTorque>
         <publishTf>1</publishTf>
         <publishOdomTf>1</publishOdomTf>
