Commit message: Added 2d nav

File: mirte_description/urdf/robot_base.gazebo.xacro (robot description, xacro)
@@ -3,4 +3,6 @@
   <xacro:property name="set_mu1" value="0.5" />
   <xacro:property name="set_mu2" value="0.5" />
+  <xacro:property name="set_kp" value="1000000" />
+  <xacro:property name="set_kd" value="10000" />
    <gazebo reference="base_link">
        <material>Gazebo/Black</material>
@@ -9,6 +11,6 @@
        <mu1>${set_mu1}</mu1>
        <mu2>${set_mu2}</mu2>
-       <!-- <kp>1000.0</kp>
-       <kd>0.1</kd>        -->
+       <kp>${set_kp}</kp>
+       <kd>${set_kd}</kd>
        <material>Gazebo/Orange</material>
    </gazebo>
@@ -16,6 +18,6 @@
        <mu1>${set_mu1}</mu1>
        <mu2>${set_mu2}</mu2>
-       <!-- <kp>1000.0</kp>
-       <kd>0.1</kd> -->
+       <kp>${set_kp}</kp>
+       <kd>${set_kd}</kd>
        <material>Gazebo/Orange</material>
    </gazebo>
@@ -23,6 +25,6 @@
        <mu1>${set_mu1}</mu1>
        <mu2>${set_mu2}</mu2>
-       <!-- <kp>1000.0</kp>
-       <kd>0.1</kd>        -->
+       <kp>${set_kp}</kp>
+       <kd>${set_kd}</kd>
        <material>Gazebo/Orange</material>
    </gazebo>
@@ -30,6 +32,6 @@
        <mu1>${set_mu1}</mu1>
        <mu2>${set_mu2}</mu2>
-       <!-- <kp>1000.0</kp>
-       <kd>0.1</kd>        -->
+       <kp>${set_kp}</kp>
+       <kd>${set_kd}</kd>
        <material>Gazebo/Orange</material>
    </gazebo>
@@ -120,5 +122,5 @@
             <legacyModeNS>false</legacyModeNS>
        </plugin>
-       <plugin name="mecanum_controller" filename="libgazebo_ros_mecanum_drive.so">
+       <!-- <plugin name="mecanum_controller" filename="libgazebo_ros_mecanum_drive.so">
             <robotNamespace>/</robotNamespace>
             <legacyMode>false</legacyMode>
@@ -139,12 +141,12 @@
             <publishWheelJointState>true</publishWheelJointState>
             <WheelTorque>1</WheelTorque>
-            <wheelAcceleration>2.8</wheelAcceleration>
+            <wheelAcceleration>2</wheelAcceleration>
             <publishTf>1</publishTf>
             <isRollerModel>true</isRollerModel>
-       </plugin>
-      <!-- <plugin name="diff_drive_controller" filename="libgazebo_ros_diff_drive.so">
+       </plugin> -->
+      <plugin name="diff_drive_controller" filename="libgazebo_ros_diff_drive.so">
         <legacyMode>false</legacyMode>
         <alwaysOn>true</alwaysOn>
-        <updateRate>50.0</updateRate>
+        <updateRate>500.0</updateRate>
         <leftJoint>front_left_wheel_joint, rear_left_wheel_joint</leftJoint>
         <rightJoint>front_right_wheel_joint, rear_right_wheel_joint</rightJoint>
@@ -158,10 +160,10 @@
         <odometryTopic>odom</odometryTopic>
         <robotBaseFrame>base_link</robotBaseFrame>
-        <wheelAcceleration>2.8</wheelAcceleration>
+        <wheelAcceleration>2</wheelAcceleration>
         <publishWheelJointState>true</publishWheelJointState>
         <publishWheelTF>false</publishWheelTF>
-        <odometrySource>world</odometrySource>
+        <odometrySource>odom</odometrySource>
         <rosDebugLevel>Debug</rosDebugLevel>
-      </plugin> -->
+      </plugin>
    </gazebo>
 </robot>
