Commit message: Added multibot

File: mirte_description/urdf/mirte_description.urdf.xacro (robot description, xacro)
@@ -49,4 +49,10 @@
     </collision>
   </link>
+  <!-- <link name="base_footprint"/>
+  <joint name="base_joint" type="fixed">
+      <parent link="base_footprint"/>
+      <child link="base_link"/>
+      <origin xyz="0 0 0.010" rpy="0 0 0"/>
+  </joint>   -->
   <link
     name="front_left_wheel_link">

File: mirte_description/urdf/robot_base.gazebo.xacro (robot description, xacro)
@@ -5,4 +5,5 @@
   <xacro:property name="set_kp" value="1000000" />
   <xacro:property name="set_kd" value="10000" />
+  <xacro:arg name="robot_tf_prefix" default=""/>
    <gazebo reference="base_link">
        <material>Gazebo/Black</material>
@@ -67,6 +68,6 @@
         </ray>
         <plugin name="lidar_sensor_controller" filename="libgazebo_ros_laser.so">
-            <topicName>/scan</topicName>
-            <frameName>lidar_link</frameName>
+            <topicName>scan</topicName>
+            <frameName>$(arg robot_tf_prefix)/lidar_link</frameName>
         </plugin>
         </sensor>
@@ -118,5 +119,5 @@
    <gazebo>
         <plugin name="gazebo_ros_control" filename="libgazebo_ros_control.so">
-            <robotNamespace>/</robotNamespace>
+            <robotNamespace>$(arg robot_tf_prefix)</robotNamespace>
             <controlPeriod>0.001</controlPeriod>
             <legacyModeNS>false</legacyModeNS>
@@ -145,24 +146,23 @@
             <isRollerModel>true</isRollerModel>
        </plugin> -->
-      <plugin name="diff_drive_controller" filename="libgazebo_ros_diff_drive.so">
+      <plugin name="$(arg robot_tf_prefix)_diff_drive_controller" filename="libgazebo_ros_diff_drive.so">
+        <commandTopic>cmd_vel</commandTopic>
+        <odometryTopic>odom</odometryTopic>
+        <odometryFrame>odom</odometryFrame>
+        <odometrySource>map</odometrySource>
+        <publishOdomTF>true</publishOdomTF>
+        <robotBaseFrame>base_link</robotBaseFrame>
+        <publishWheelTF>false</publishWheelTF>
+        <publishTf>true</publishTf>
+        <publishWheelJointState>true</publishWheelJointState>
         <legacyMode>false</legacyMode>
-        <alwaysOn>true</alwaysOn>
-        <updateRate>500.0</updateRate>
+        <updateRate>50</updateRate>
         <leftJoint>front_left_wheel_joint, rear_left_wheel_joint</leftJoint>
         <rightJoint>front_right_wheel_joint, rear_right_wheel_joint</rightJoint>
         <wheelSeparation>0.256</wheelSeparation>
         <wheelDiameter>0.102</wheelDiameter>
-        <wheelTorque>1</wheelTorque>
-        <publishTf>1</publishTf>
-        <publishOdomTf>1</publishOdomTf>
-        <odometryFrame>map</odometryFrame>
-        <commandTopic>cmd_vel</commandTopic>
-        <odometryTopic>odom</odometryTopic>
-        <robotBaseFrame>base_link</robotBaseFrame>
-        <wheelAcceleration>2</wheelAcceleration>
-        <publishWheelJointState>true</publishWheelJointState>
-        <publishWheelTF>false</publishWheelTF>
-        <odometrySource>odom</odometrySource>
-        <rosDebugLevel>Debug</rosDebugLevel>
+        <wheelAcceleration>1</wheelAcceleration>
+        <wheelTorque>10</wheelTorque>
+        <rosDebugLevel>na</rosDebugLevel>
       </plugin>
    </gazebo>
